Commit message: project 2 finished ch-6

File: go_chase_it/catkin_ws/src/my_robot/urdf/my_robot.xacro (robot description, xacro)
@@ -64,39 +64,7 @@
   </joint>
   <link name = 'left_wheel'>
-    <!--<inertial>
+        <inertial>
       <mass value="5"/>
-      <origin xyz = "0 0 0 0" rpy="0 1.5707 1.5707"/>
-        <inertia
-          ixx="0.1" ixy="0" ixz="0"
-          iyy="0.1" iyz="0"
-          izz="0.1"
-        />
-    </inertial> -->
-    <collision>
-        <origin xyz = "0 0 0 0" rpy="0 1.5707 1.5707"/>
-        <geometry>
-            <cylinder radius = "0.1" length = "0.05"/>
-        </geometry>
-    </collision>
-    <visual>
-        <origin xyz = "0 0 0 0" rpy="0 1.5707 1.5707"/>
-        <geometry>
-            <cylinder radius = "0.1" length = "0.05"/>
-        </geometry>
-    </visual>
-  </link>
-  <!-- <joint type="continuous" name="right_wheel_hinge">
-    <origin xyz="0 0.15 0" rpy="0 0 0"/>
-    <child link="right_wheel"/>
-    <parent link="chassis"/>
-    <axis xyz="0 1 0" rpy="0 0 0"/>
-    <limit effort="10000" velocity="1000"/>
-    <dynamics damping="1.0" friction="1.0"/>
-  </joint>
-<link name = 'right_wheel'>
-    <pose>0 0 0.1 0 0 0</pose>
-    <inertial>
-      <mass value="5"/>
-      <origin xyz = "0 0 0 0" rpy="0 1.5707 1.5707"/>
+      <origin xyz = "0 0 0" rpy="0 1.5707 1.5707"/>
         <inertia
           ixx="0.1" ixy="0" ixz="0"
@@ -106,11 +74,5 @@
     </inertial>
     <collision>
-        <origin xyz = "0 0 0 0" rpy="0 1.5707 1.5707"/>
-        <geometry>
-            <cylinder radius = "0.1" length = "0.05"/>
-        </geometry>
-    </collision>
-    <collision>
-        <origin xyz = "0 0 0 0" rpy="0 1.5707 1.5707"/>
+        <origin xyz = "0 0 0" rpy="0 1.5707 1.5707"/>
         <geometry>
             <cylinder radius = "0.1" length = "0.05"/>
@@ -118,9 +80,40 @@
     </collision>
     <visual>
-        <origin xyz = "0 0 0 0" rpy="0 1.5707 1.5707"/>
+        <origin xyz = "0 0 0" rpy="0 1.5707 1.5707"/>
         <geometry>
             <cylinder radius = "0.1" length = "0.05"/>
         </geometry>
     </visual>
-  </link> -->
+  </link>
+<joint type="continuous" name="right_wheel_hinge">
+    <origin xyz="0 -0.15 0" rpy="0 0 0"/>
+    <child link="right_wheel"/>
+    <parent link="chassis"/>
+    <axis xyz="0 1 0" rpy="0 0 0"/>
+    <limit effort="10000" velocity="1000"/>
+    <dynamics damping="1.0" friction="1.0"/>
+  </joint>
+  <link name = 'right_wheel'>
+        <inertial>
+      <mass value="5"/>
+      <origin xyz = "0 0 0" rpy="0 1.5707 1.5707"/>
+        <inertia
+          ixx="0.1" ixy="0" ixz="0"
+          iyy="0.1" iyz="0"
+          izz="0.1"
+        />
+    </inertial>
+    <collision>
+        <origin xyz = "0 0 0" rpy="0 1.5707 1.5707"/>
+        <geometry>
+            <cylinder radius = "0.1" length = "0.05"/>
+        </geometry>
+    </collision>
+    <visual>
+        <origin xyz = "0 0 0" rpy="0 1.5707 1.5707"/>
+        <geometry>
+            <cylinder radius = "0.1" length = "0.05"/>
+        </geometry>
+    </visual>
+  </link>
 </robot>

Commit message: added a camera in urdf file

File: go_chase_it/catkin_ws/src/my_robot/urdf/my_robot.xacro (robot description, xacro)
@@ -117,3 +117,37 @@
     </visual>
   </link>
+  <!-- make a fixed joint between chassis and camera-->
+  <joint type="fixed" name="camera_joint">
+    <origin xyz="0.2 0 0" rpy="0 0 0"/>
+    <axis xyz="0 1 0"/>
+    <child link="camera"/>
+    <parent link="chassis"/>
+  </joint>
+  <link name ="camera">
+    <origin xyz="0 0 0" rpy="0 0 0"/>
+    <geometry>
+      <box size="0.05 0.05 0.05"/>
+    </geometry>
+    <inertial>
+      <mass value="0.1"/>
+      <origin xyz="0 0 0" rpy="0 0 0"/>
+      <inertia
+        ixx="1e-6" ixy="0" ixz="0"
+        iyy="1e-6" iyz="0"
+        izz="1e-6"
+        />
+    </inertial>
+    <collision>
+      <origin xyz="0 0 0" rpy="0 0 0"/>
+      <geometry>
+        <box size="0.05 0.05 0.05"/>
+      </geometry>
+    </collision>
+    <visual>
+      <origin xyz="0 0 0" rpy="0 0 0"/>
+      <geometry>
+        <box size="0.05 0.05 0.05"/>
+      </geometry>
+    </visual>
+  </link>
 </robot>

Commit message: Added Lidar

File: go_chase_it/catkin_ws/src/my_robot/urdf/my_robot.xacro (robot description, xacro)
@@ -151,3 +151,31 @@
     </visual>
   </link>
+  <joint>
+  </joint>
+  <!-- make a joint named hukuyo_joint with chassis as a parent and hokuyu as a child-->
+  <joint type="fixed" name="hokuyo_joint">
+    <origin xyz="0.15 0 0.1" rpy="0 0 0"/>
+    <axis xyz="0 1 0"/>
+    <child link="hokuyo"/>
+    <parent link="chassis"/>
+  </joint>
+  <link name ="hokuyo">
+    <origin xyz="0 0 0" rpy="0 0 0"/>
+    <visual>
+      <geometry filename= "package://my_robot/meshes/hokuyo.dae"/>
+    <visual/>
+    <collision>
+      <origin xyz="0 0 0" rpy="0 0 0"/>
+      <geometry>
+        <box size="0.1 0.1 0.1"/>
+      </geometry>
+    </collision>
+    <inertial>
+      <mass value="1e-5"/>
+      <inertia
+        ixx="1e-6" ixy="0" ixz="0"
+        iyy="1e-6" iyz="0"
+        izz="1e-6"
+        />
+    </inertial>
 </robot>

Commit message: added Lidar Sensor

File: go_chase_it/catkin_ws/src/my_robot/urdf/my_robot.xacro (robot description, xacro)
@@ -1,4 +1,17 @@
 <?xml version='1.0'?>
+<xacro  :include filename="$(find my_robot)/urfd/my_robot.gazebo"/>
 <robot name="my_robot" xmlns:xacro="http://www.ros.org/wiki/xacro">
+<gazebo reference = "left_wheel">
+  <material>Gazebo/Green</material>
+</gazebo>
+<gazebo reference = "right_wheel">
+  <material>Gazebo/Green</material>
+</gazebo>
+<gazebo reference = "chassis">
+  <material>Gazebo/Blue</material>
+</gazebo>
+<gazebo reference = "camera">
+  <material>Gazebo/Red</material>
+</gazebo>
   <link name="robot_footprint"></link>
   <joint name="robot_footprint_joint" type="fixed">
@@ -117,6 +130,5 @@
     </visual>
   </link>
-  <!-- make a fixed joint between chassis and camera-->
-  <joint type="fixed" name="camera_joint">
+    <joint type="fixed" name="camera_joint">
     <origin xyz="0.2 0 0" rpy="0 0 0"/>
     <axis xyz="0 1 0"/>
@@ -151,7 +163,4 @@
     </visual>
   </link>
-  <joint>
-  </joint>
-  <!-- make a joint named hukuyo_joint with chassis as a parent and hokuyu as a child-->
   <joint type="fixed" name="hokuyo_joint">
     <origin xyz="0.15 0 0.1" rpy="0 0 0"/>
@@ -160,9 +169,13 @@
     <parent link="chassis"/>
   </joint>
-  <link name ="hokuyo">
+<link name ="hokuyo">
     <origin xyz="0 0 0" rpy="0 0 0"/>
     <visual>
-      <geometry filename= "package://my_robot/meshes/hokuyo.dae"/>
-    <visual/>
+    <origin xyz="0 0 0" rpy="0 0 0"/>
+      <geometry><mesh filename= "package://my_robot/meshes/hokuyo.dae"/></geometry>
+    <!-- <geometry>
+        <box size="0.1 0.1 0.1"/>
+      </geometry> -->
+    </visual>
     <collision>
       <origin xyz="0 0 0" rpy="0 0 0"/>
@@ -179,3 +192,4 @@
         />
     </inertial>
+  </link>
 </robot>

Commit message: fixed the weird xacro:include bug

File: go_chase_it/catkin_ws/src/my_robot/urdf/my_robot.xacro (robot description, xacro)
@@ -1,4 +1,3 @@
 <?xml version='1.0'?>
-<xacro:include filename="$(find my_robot)/urdf/my_robot.gazebo" />
 <robot name="my_robot" xmlns:xacro="http://www.ros.org/wiki/xacro">
 <gazebo reference = "left_wheel">
@@ -14,4 +13,5 @@
   <material>Gazebo/Red</material>
 </gazebo>
+<xacro:include filename="$(find my_robot)/urdf/my_robot.gazebo" />
   <link name="robot_footprint"></link>
   <joint name="robot_footprint_joint" type="fixed">
@@ -174,7 +174,4 @@
     <origin xyz="0 0 0" rpy="0 0 0"/>
       <geometry><mesh filename= "package://my_robot/meshes/hokuyo.dae"/></geometry>
-    <!-- <geometry>
-        <box size="0.1 0.1 0.1"/>
-      </geometry> -->
     </visual>
     <collision>

Commit message: Fixing the project review comments

File: go_chase_it/catkin_ws/src/my_robot/urdf/my_robot.xacro (robot description, xacro)
@@ -24,5 +24,5 @@
     <inertial>
       <mass value="15.0"/>
-      <origin xyz="0.0 0 0" rpy=" 0 0 0"/>
+      <origin xyz="0 0 0" rpy=" 0 0 0"/>
       <inertia
           ixx="0.1" ixy="0" ixz="0"
@@ -35,4 +35,5 @@
       <geometry>
         <box size=".4 .2 .1"/>
+	<!--<cylinder radius ="0.1" length="0.1"/>-->
       </geometry>
     </collision>
@@ -41,4 +42,5 @@
       <geometry>
         <box size=".4 .2 .1"/>
+	<!--<cylinder radius ="0.1" length="0.1"/>-->
       </geometry>
     </visual>

Commit message: Modified the robot dimensions and colours according to the project review

File: go_chase_it/catkin_ws/src/my_robot/urdf/my_robot.xacro (robot description, xacro)
@@ -2,14 +2,14 @@
 <robot name="my_robot" xmlns:xacro="http://www.ros.org/wiki/xacro">
 <gazebo reference = "left_wheel">
-  <material>Gazebo/Green</material>
+  <material>Gazebo/DarkGrey</material>
 </gazebo>
 <gazebo reference = "right_wheel">
-  <material>Gazebo/Green</material>
+  <material>Gazebo/DarkGrey</material>
 </gazebo>
 <gazebo reference = "chassis">
-  <material>Gazebo/Blue</material>
+  <material>Gazebo/Orange</material>
 </gazebo>
 <gazebo reference = "camera">
-  <material>Gazebo/Red</material>
+  <material>Gazebo/Purple</material>
 </gazebo>
 <xacro:include filename="$(find my_robot)/urdf/my_robot.gazebo" />
@@ -23,5 +23,5 @@
     <pose>0 0 0.1 0 0 0</pose>
     <inertial>
-      <mass value="15.0"/>
+      <mass value="1.0"/>
       <origin xyz="0 0 0" rpy=" 0 0 0"/>
       <inertia
@@ -34,6 +34,6 @@
       <origin xyz="0 0 0" rpy=" 0 0 0"/>
       <geometry>
-        <box size=".4 .2 .1"/>
-	<!--<cylinder radius ="0.1" length="0.1"/>-->
+        <box size=".8 .2 .1"/>
+	<!--<cylinder radius ="0.2" length="0.1"/>-->
       </geometry>
     </collision>
@@ -41,10 +41,10 @@
       <origin xyz="0 0 0" rpy=" 0 0 0"/>
       <geometry>
-        <box size=".4 .2 .1"/>
-	<!--<cylinder radius ="0.1" length="0.1"/>-->
+        <box size=".8 .2 .1"/>
+	<!--<cylinder radius ="0.2" length="0.1"/>-->
       </geometry>
     </visual>
-    <collision name='back_caster_collision'>
-      <origin xyz="-0.15 0 -0.05" rpy=" 0 0 0"/>
+   <collision name='back_caster_collision'>
+      <origin xyz="-0.3 0 -0.025" rpy=" 0 0 0"/>
       <geometry>
         <sphere radius="0.0499"/>
@@ -52,5 +52,5 @@
     </collision>
     <visual name='back_caster_visual'>
-      <origin xyz="-0.15 0 -0.05" rpy=" 0 0 0"/>
+      <origin xyz="-0.3 0 -0.05" rpy=" 0 0 0"/>
       <geometry>
         <sphere radius="0.05"/>
@@ -58,11 +58,11 @@
     </visual>
     <collision name='front_caster_collision'>
-      <origin xyz="0.15 0 -0.05" rpy=" 0 0 0"/>
+      <origin xyz="0.3 0 -0.025" rpy=" 0 0 0"/>
       <geometry>
         <sphere radius="0.0499"/>
       </geometry>
-    </collision>
+    </collision> -->
     <visual name='front_caster_visual'>
-      <origin xyz="0.15 0 -0.05" rpy=" 0 0 0"/>
+      <origin xyz="0.3 0 -0.025" rpy=" 0 0 0"/>
       <geometry>
         <sphere radius="0.05"/>
@@ -71,5 +71,5 @@
   </link>
   <joint type="continuous" name="left_wheel_hinge">
-    <origin xyz="0 0.15 0" rpy="0 0 0"/>
+    <origin xyz="-0.3 0.15 0" rpy="0 0 0"/>
     <child link="left_wheel"/>
     <parent link="chassis"/>
@@ -91,5 +91,5 @@
         <origin xyz = "0 0 0" rpy="0 1.5707 1.5707"/>
         <geometry>
-            <cylinder radius = "0.1" length = "0.05"/>
+            <cylinder radius = "0.075" length = "0.05"/>
         </geometry>
     </collision>
@@ -97,10 +97,10 @@
         <origin xyz = "0 0 0" rpy="0 1.5707 1.5707"/>
         <geometry>
-            <cylinder radius = "0.1" length = "0.05"/>
+            <cylinder radius = "0.075" length = "0.05"/>
         </geometry>
     </visual>
   </link>
 <joint type="continuous" name="right_wheel_hinge">
-    <origin xyz="0 -0.15 0" rpy="0 0 0"/>
+    <origin xyz="-0.3 -0.15 0" rpy="0 0 0"/>
     <child link="right_wheel"/>
     <parent link="chassis"/>
@@ -122,5 +122,5 @@
         <origin xyz = "0 0 0" rpy="0 1.5707 1.5707"/>
         <geometry>
-            <cylinder radius = "0.1" length = "0.05"/>
+            <cylinder radius = "0.075" length = "0.05"/>
         </geometry>
     </collision>
@@ -128,10 +128,10 @@
         <origin xyz = "0 0 0" rpy="0 1.5707 1.5707"/>
         <geometry>
-            <cylinder radius = "0.1" length = "0.05"/>
+            <cylinder radius = "0.075" length = "0.05"/>
         </geometry>
     </visual>
   </link>
-    <joint type="fixed" name="camera_joint">
-    <origin xyz="0.2 0 0" rpy="0 0 0"/>
+  <joint type="fixed" name="camera_joint">
+    <origin xyz="0.4 0 0" rpy="0 0 0"/>
     <axis xyz="0 1 0"/>
     <child link="camera"/>
@@ -166,5 +166,5 @@
   </link>
   <joint type="fixed" name="hokuyo_joint">
-    <origin xyz="0.15 0 0.1" rpy="0 0 0"/>
+    <origin xyz="0.35 0 0.1" rpy="0 0 0"/>
     <axis xyz="0 1 0"/>
     <child link="hokuyo"/>
